File: v2/Appletini_board/bus_transceivers.kicad_sch (KiCad schematic)
At the start: 17 parts, among them U1 SN74LVC543ADW, U10 SN74LVC543ADW, U14 74AHC1G126, U4 SN74LVC543ADW, U5 TXS0108EPW, U6 74LS08, U7 74AHC1G126, U9 SN74LVC543ADW

Commit message: v2 board first draft done
Parts:
- added R3: 10K, Resistor_SMD:R_0402_1005Metric, symbol Device:R_US
- added U8: SN74LVC1G14DBV, Package_TO_SOT_SMD:SOT-23-5, symbol 74xGxx:SN74LVC1G14DBV
Connections:
- net +3.3V: now also U8.5 (VCC)
- net BUS_~{ENABLE}: now also U8.2
- net GND: now also R3.2, U8.3 (GND)
- net LEVEL_ENABLE: now also R3.1, U8.4
Other:
- moved on the sheet: C1, U6A, U6B, U6C, U6D, U6E

Commit message: fixes
Parts:
- removed C1: 100pF, Capacitor_SMD:C_1206_3216Metric, symbol Device:C
- removed U6: 74LS08, Package_SO:TSSOP-14_4.4x5mm_P0.65mm, symbol 74xx:74LS08
- added C13, C14: 100pF, Capacitor_SMD:C_1206_3216Metric, symbol Device:C
- added R2, R6: 10K, Resistor_SMD:R_0402_1005Metric, symbol Device:R_US
- added U13: 74LVC1G08, Package_TO_SOT_SMD:SOT-353_SC-70-5, symbol 74xGxx:74LVC1G08
- added U8: 74LCX07, Package_SO:TSSOP-14_4.4x5mm_P0.65mm, symbol 74xx:74LCX07
- renumbered C7 to C10, C23 to C11, C22 to C12, C8 to C5, C9 to C6, C10 to C7, C11 to C8, C2 to C9, R3 to R5, U7 to U10, U8 to U11, U1 to U3, U10 to U5, U9 to U6, U5 to U7, U14 to U9
Connections:
- net +3.3V: now also C13.1, C14.1, R2.1, R6.1, U13.5 (VCC), U8.14 (VCC)
- net BUS_~{DMAIN}: now also U13.1, U8.9
- net BUS_~{INTIN}: now also U8.1
- net GND: now also C13.2, C14.2, U13.3 (GND), U8.13, U8.7 (GND)
- net TEENSY_REQ_DMA: now also U13.2
- net TEENSY_REQ_~{DMAOUT}: now also R6.2, U8.11
- net CTRL_~{DMAOUT} renamed ~{DMAOUT}
- net ~{DMAOUT}: now also U8.10, U8.8
- net CTRL_~{INTOUT} renamed ~{INTOUT}
- net ~{INTOUT}: now also U8.2, U8.6
- net PICO_CTRL_~{DMA} renamed ~{DMA}
- net PICO_CTRL_~{INH} renamed ~{INH}
- net PICO_CTRL_~{RDY} renamed ~{RDY}
- net TEENSY_CTRL_~{IRQ} renamed ~{IRQ}
- net ~{IRQ}: now also U8.4
- new net DMA_CYCLE_ACTIVE: U13.4
- new net TEENSY_REQ_~{IRQ}: R2.2, U8.3, U8.5
Other:
- moved on the sheet: R5, U11

Commit message: checkpoint before lvc573 rework
Parts:
- C10, C11, C12, C13, C14, C5, C6, C7, C8, C9: value 100pF -> 100nF; LCSC (none) -> C24497
- R2, R5, R6: LCSC (none) -> C2991755
- U10, U9: footprint Package_TO_SOT_SMD:SOT-353_SC-70-5 -> Package_TO_SOT_SMD:SOT-23-5; LCSC (none) -> C7834
- U11: LCSC (none) -> C7835
- U13: footprint Package_TO_SOT_SMD:SOT-353_SC-70-5 -> Package_TO_SOT_SMD:SOT-23-5; LCSC (none) -> C7666
- U3, U4, U5, U6: LCSC (none) -> C2676536
- U7: LCSC (none) -> C17206
- U8: LCSC (none) -> C7809
Changed lines of the file:
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@@
       (effects (font (size 1.27 1.27)))
     )
-    (property "Footprint" "Package_TO_SOT_SMD:SOT-353_SC-70-5" (at 247.65 109.22 0)
+    (property "Footprint" "Package_TO_SOT_SMD:SOT-23-5" (at 247.65 109.22 0)
       (effects (font (size 1.27 1.27)) hide)
     )
     (property "Datasheet" "https://www.ti.com/lit/ds/symlink/sn74lvc1g08.pdf" (at 247.65 109.22 0)
+      (effects (font (size 1.27 1.27)) hide)
+    )
+    (property "LCSC" "C7666" (at 247.65 109.22 0)
       (effects (font (size 1.27 1.27)) hide)
     )
@@
     )
     (property "Datasheet" "~" (at 210.82 40.64 0)
+      (effects (font (size 1.27 1.27)) hide)
+    )
+    (property "LCSC" "C2991755" (at 210.82 40.64 0)
       (effects (font (size 1.27 1.27)) hide)
     )
@@
     (property "Datasheet" "SN74LVC543ADW" (at 59.69 25.4 0)
       (effects (font (size 1.27 1.27) italic) hide)
+    )
+    (property "LCSC" "C2676536" (at 59.69 25.4 0)
+      (effects (font (size 1.27 1.27)) hide)
     )
     (pin "1")
@@
       (effects (font (size 1.27 1.27)) (justify left))
     )
-    (property "Value" "100pF" (at 118.11 93.345 0)
+    (property "Value" "100nF" (at 118.11 93.345 0)
       (effects (font (size 1.27 1.27)) (justify left))
     )
@@
       (effects (font (size 1.27 1.27)) hide)
     )
+    (property "LCSC" "C24497" (at 114.3 91.44 0)
+      (effects (font (size 1.27 1.27)) hide)
+    )
     (pin "1")
     (pin "2")
@@
       (effects (font (size 1.27 1.27)) (justify left))
     )
-    (property "Value" "100pF" (at 179.07 53.975 0)
+    (property "Value" "100nF" (at 179.07 53.975 0)
       (effects (font (size 1.27 1.27)) (justify left))
     )
@@
     )
     (property "Datasheet" "~" (at 175.26 52.07 0)
+      (effects (font (size 1.27 1.27)) hide)
+    )
+    (property "LCSC" "C24497" (at 175.26 52.07 0)
       (effects (font (size 1.27 1.27)) hide)
     )
@@
       (effects (font (size 1.27 1.27)) (justify left))
     )
-    (property "Value" "100pF" (at 20.32 102.235 0)
+    (property "Value" "100nF" (at 20.32 102.235 0)
       (effects (font (size 1.27 1.27)) (justify left))
     )
@@
     )
     (property "Datasheet" "~" (at 16.51 100.33 0)
+      (effects (font (size 1.27 1.27)) hide)
+    )
+    (property "LCSC" "C24497" (at 16.51 100.33 0)
       (effects (font (size 1.27 1.27)) hide)
     )
@@
     )
     (property "Datasheet" "www.st.com/resource/en/datasheet/74lcx07.pdf" (at 224.79 27.94 0)
+      (effects (font (size 1.27 1.27)) hide)
+    )
+    (property "LCSC" "C7809" (at 224.79 27.94 0)
       (effects (font (size 1.27 1.27)) hide)
     )
@@
       (effects (font (size 1.27 1.27)) (justify left))
     )
-    (property "Value" "100pF" (at 110.49 55.245 0)
+    (property "Value" "100nF" (at 110.49 55.245 0)
       (effects (font (size 1.27 1.27)) (justify left))
     )
@@
       (effects (font (size 1.27 1.27)) hide)
     )
+    (property "LCSC" "C24497" (at 106.68 53.34 0)
+      (effects (font (size 1.27 1.27)) hide)
+    )
     (pin "1")
     (pin "2")
@@
     )
     (property "Datasheet" "http://www.ti.com/lit/ds/symlink/sn74lvc1g14.pdf" (at 237.49 144.78 0)
+      (effects (font (size 1.27 1.27)) hide)
+    )
+    (property "LCSC" "C7835" (at 237.49 144.78 0)
       (effects (font (size 1.27 1.27)) hide)
     )
@@
       (effects (font (size 1.27 1.27)) (justify left))
     )
-    (property "Value" "100pF" (at 278.13 33.655 0)
+    (property "Value" "100nF" (at 278.13 33.655 0)
       (effects (font (size 1.27 1.27)) (justify left))
     )
@@
     )
     (property "Datasheet" "~" (at 274.32 31.75 0)
+      (effects (font (size 1.27 1.27)) hide)
+    )
+    (property "LCSC" "C24497" (at 274.32 31.75 0)
       (effects (font (size 1.27 1.27)) hide)
     )
@@
       (effects (font (size 1.27 1.27)) (justify left))
     )
-    (property "Value" "100pF" (at 22.86 167.005 0)
+    (property "Value" "100nF" (at 22.86 167.005 0)
       (effects (font (size 1.27 1.27)) (justify left))
     )
@@
     )
     (property "Datasheet" "~" (at 19.05 165.1 0)
+      (effects (font (size 1.27 1.27)) hide)
+    )
+    (property "LCSC" "C24497" (at 19.05 165.1 0)
       (effects (font (size 1.27 1.27)) hide)
     )
@@
     (property "Datasheet" "SN74LVC543ADW" (at 152.4 128.27 0)
       (effects (font (size 1.27 1.27) italic) hide)
+    )
+    (property "LCSC" "C2676536" (at 152.4 128.27 0)
+      (effects (font (size 1.27 1.27)) hide)
     )
     (pin "1")
@@
       (effects (font (size 1.27 1.27)) (justify left))
     )
-    (property "Value" "100pF" (at 175.26 92.075 0)
+    (property "Value" "100nF" (at 175.26 92.075 0)
       (effects (font (size 1.27 1.27)) (justify left))
     )
@@
       (effects (font (size 1.27 1.27)) hide)
     )
+    (property "LCSC" "C24497" (at 171.45 90.17 0)
+      (effects (font (size 1.27 1.27)) hide)
+    )
     (pin "1")
     (pin "2")
@@
     )
     (property "Datasheet" "www.st.com/resource/en/datasheet/74lcx07.pdf" (at 256.54 31.75 0)
+      (effects (font (size 1.27 1.27)) hide)
+    )
+    (property "LCSC" "C7809" (at 256.54 31.75 0)
       (effects (font (size 1.27 1.27)) hide)
     )
@@
       (effects (font (size 1.27 1.27)))
     )
-    (property "Footprint" "Package_TO_SOT_SMD:SOT-353_SC-70-5" (at 189.23 99.06 0)
+    (property "Footprint" "Package_TO_SOT_SMD:SOT-23-5" (at 189.23 99.06 0)
       (effects (font (size 1.27 1.27)) hide)
     )
     (property "Datasheet" "http://www.ti.com/lit/sg/scyt129e/scyt129e.pdf" (at 189.23 99.06 0)
+      (effects (font (size 1.27 1.27)) hide)
+    )
+    (property "LCSC" "C7834" (at 189.23 99.06 0)
       (effects (font (size 1.27 1.27)) hide)
     )
@@
     )
     (property "Datasheet" "www.ti.com/lit/ds/symlink/txs0108e.pdf" (at 140.97 57.15 0)
+      (effects (font (size 1.27 1.27)) hide)
+    )
+    (property "LCSC" "C17206" (at 140.97 54.61 0)
       (effects (font (size 1.27 1.27)) hide)
     )
@@
     )
     (property "Datasheet" "www.st.com/resource/en/datasheet/74lcx07.pdf" (at 266.7 73.66 0)
+      (effects (font (size 1.27 1.27)) hide)
+    )
+    (property "LCSC" "C7809" (at 266.7 73.66 0)
       (effects (font (size 1.27 1.27)) hide)
     )
@@
       (effects (font (size 1.27 1.27)) (justify left))
     )
-    (property "Value" "100pF" (at 237.49 99.695 0)
+    (property "Value" "100nF" (at 237.49 99.695 0)
       (effects (font (size 1.27 1.27)) (justify left))
     )
@@
     )
     (property "Datasheet" "~" (at 233.68 97.79 0)
+      (effects (font (size 1.27 1.27)) hide)
+    )
+    (property "LCSC" "C24497" (at 233.68 97.79 0)
       (effects (font (size 1.27 1.27)) hide)
     )
@@
     (property "Datasheet" "SN74LVC543ADW" (at 59.69 88.9 0)
       (effects (font (size 1.27 1.27) italic) hide)
+    )
+    (property "LCSC" "C2676536" (at 59.69 88.9 0)
+      (effects (font (size 1.27 1.27)) hide)
     )
     (pin "1")
@@
       (effects (font (size 1.27 1.27)) hide)
     )
+    (property "LCSC" "C7809" (at 224.79 58.42 0)
+      (effects (font (size 1.27 1.27)) hide)
+    )
     (pin "1")
     (pin "2")
@@
       (effects (font (size 1.27 1.27)) hide)
     )
+    (property "LCSC" "C2991755" (at 261.62 153.67 0)
+      (effects (font (size 1.27 1.27)) hide)
+    )
     (pin "1")
     (pin "2")
@@
     )
     (property "Datasheet" "~" (at 212.09 71.12 0)
+      (effects (font (size 1.27 1.27)) hide)
+    )
+    (property "LCSC" "C2991755" (at 212.09 71.12 0)
       (effects (font (size 1.27 1.27)) hide)
     )
@@
       (effects (font (size 1.27 1.27)) (justify left))
     )
-    (property "Value" "100pF" (at 20.32 38.735 0)
+    (property "Value" "100nF" (at 20.32 38.735 0)
       (effects (font (size 1.27 1.27)) (justify left))
     )
@@
       (effects (font (size 1.27 1.27)) hide)
     )
+    (property "LCSC" "C24497" (at 16.51 36.83 0)
+      (effects (font (size 1.27 1.27)) hide)
+    )
+    (property "Field5" "" (at 16.51 36.83 0)
+      (effects (font (size 1.27 1.27)) hide)
+    )
+    (property "Field6" "" (at 16.51 36.83 0)
+      (effects (font (size 1.27 1.27)) hide)
+    )
     (pin "1")
     (pin "2")
@@
     )
     (property "Datasheet" "www.st.com/resource/en/datasheet/74lcx07.pdf" (at 224.79 44.45 0)
+      (effects (font (size 1.27 1.27)) hide)
+    )
+    (property "LCSC" "C7809" (at 224.79 44.45 0)
       (effects (font (size 1.27 1.27)) hide)
     )
@@
       (effects (font (size 1.27 1.27)))
     )
-    (property "Footprint" "Package_TO_SOT_SMD:SOT-353_SC-70-5" (at 133.35 100.33 0)
+    (property "Footprint" "Package_TO_SOT_SMD:SOT-23-5" (at 133.35 100.33 0)
       (effects (font (size 1.27 1.27)) hide)
     )
     (property "Datasheet" "http://www.ti.com/lit/sg/scyt129e/scyt129e.pdf" (at 133.35 100.33 0)
+      (effects (font (size 1.27 1.27)) hide)
+    )
+    (property "LCSC" "C7834" (at 133.35 100.33 0)
       (effects (font (size 1.27 1.27)) hide)
     )
@@
       (effects (font (size 1.27 1.27)) (justify left))
     )
-    (property "Value" "100pF" (at 110.49 141.605 0)
+    (property "Value" "100nF" (at 110.49 141.605 0)
       (effects (font (size 1.27 1.27)) (justify left))
     )
@@
       (effects (font (size 1.27 1.27)) hide)
     )
+    (property "LCSC" "C24497" (at 106.68 139.7 0)
+      (effects (font (size 1.27 1.27)) hide)
+    )
     (pin "1")
     (pin "2")
@@
     )
     (property "Datasheet" "www.st.com/resource/en/datasheet/74lcx07.pdf" (at 224.79 87.63 0)
+      (effects (font (size 1.27 1.27)) hide)
+    )
+    (property "LCSC" "C7809" (at 224.79 87.63 0)
       (effects (font (size 1.27 1.27)) hide)
     )
@@
       (effects (font (size 1.27 1.27)) hide)
     )
+    (property "LCSC" "C7809" (at 224.79 74.93 0)
+      (effects (font (size 1.27 1.27)) hide)
+    )
     (pin "1")
     (pin "2")
@@
       (effects (font (size 1.27 1.27) italic) hide)
     )
-    (pin "1")
+    (property "LCSC" "C2676536" (at 59.69 152.4 0)
+      (effects (font (size 1.27 1.27)) hide)
+    )
+    (pin "1")
