File: v5/AppleTini_board/AppleTini_board.kicad_pcb (KiCad board)
At the start: 4 copper layers, 101.6 x 69.8 mm, 39 parts, among them J1 Conn_02x25_Counter_Clockwise, J2 Conn_02x14_Odd_Even, J3 Conn_02x14_Odd_Even, J4 Conn_02x05_Odd_Even, J5 Conn_02x05_Odd_Even, U1 MC74LCX16245DT, U2 MC74LCX16245DT, U3 MC74LCX16245DT, U7 74LCX07, U8 74LVC1G04

Commit message: wip, reworking
Parts:
- removed C11, C12, C14, C16: C, Capacitor_SMD:C_0603_1608Metric
- removed R10, R2, R3, R4, R5, R6: R_US, Resistor_SMD:R_0402_1005Metric
- added D1: D_Schottky, Diode_SMD:Nexperia_CFP3_SOD-123W, F.Cu at (225.0, 115.2)
- added R13: R_US, Resistor_SMD:R_0402_1005Metric, F.Cu at (205.5, 95.2)
- added R14: R_US, Resistor_SMD:R_0402_1005Metric, F.Cu at (205.5, 99.0)
- added R15: R_US, Resistor_SMD:R_0402_1005Metric, F.Cu at (205.5, 102.8)
- added R16: R_US, Resistor_SMD:R_0402_1005Metric, F.Cu at (220.0, 102.8)
- added R17: R_US, Resistor_SMD:R_0402_1005Metric, F.Cu at (220.0, 99.0)
- added R18: R_US, Resistor_SMD:R_0402_1005Metric, F.Cu at (219.8, 95.2)
- added U4: 74LCX07, Package_SO:TSSOP-14_4.4x5mm_P0.65mm, F.Cu at (210.5, 78.0)
- moved C6 83.8 mm to (219.0, 75.0), turned to 0 degrees
- moved C7 73.8 mm to (216.5, 92.0), turned to 0 degrees
- moved R11 31.7 mm to (203.0, 76.2), turned to 0 degrees
- moved R12 25.4 mm to (203.0, 81.0), turned to 0 degrees
- moved R1 16.6 mm to (217.0, 78.8), turned to 180 degrees
- moved C10 6.54 mm to (182.2, 120.5)
- moved C13 6.15 mm to (193.8, 119.0)
- moved U2 6.02 mm to (173.0, 120.5)
- moved C15 5.94 mm to (212.2, 119.0)
- moved C9 5.83 mm to (163.5, 120.2)
- moved U3 5.55 mm to (203.0, 118.8)
- moved J2 4.02 mm to (157.6, 105.7)
- moved J3 4.02 mm to (157.6, 100.7)
- moved J4 4.02 mm to (157.6, 93.0)
- moved J5 4.02 mm to (157.6, 88.0)
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Connections:
- C6 pad 1: +3V3 -> +5V
- C7 pad 1: +3V3 -> +5V
- J1 pad 21: unconnected-(J1-Pin_21-Pad21) -> /BUS_~{RDY}
- J1 pad 29: unconnected-(J1-Pin_29-Pad29) -> /BUS_~{NMI}
- R1 pad 1: +3V3 -> +5V
- R1 pad 2: /B5 -> /~{OE}
- R11 pad 1: +3V3 -> +5V
- R11 pad 2: /BUS_~{INTOUT} -> /BUS_~{DMAOUT}
- R12 pad 1: +3V3 -> +5V
- R12 pad 2: /BUS_~{DMAOUT} -> /BUS_~{INTOUT}
- U1 pad 25: /A37 -> /~{OE}
- U1 pad 48: /A37 -> /~{OE}
- U2 pad 25: /A37 -> /~{OE}
- U2 pad 48: /A37 -> /~{OE}
- U3 pad 25: /A37 -> /~{OE}
- U3 pad 48: /A37 -> /~{OE}
- U7 pad 10: /BUS_~{INTOUT} -> /BUS_~{NMI}
- U7 pad 12: /BUS_~{DMAOUT} -> /BUS_~{RDY}
- U7 pad 14: +3V3 -> +5V
Routing:
- net +3V3: track 140.2 -> 0.00 mm, vias 19 -> 0
- net GND: track 128.4 -> 0.00 mm, vias 18 -> 0
- net /A37: track 121.3 -> 0.00 mm, vias 6 -> 0
- net /C49: track 110.8 -> 0.00 mm, vias 3 -> 0
- net /BUS_~{DMA}: track 68.2 -> 0.00 mm, vias 2 -> 0
- net /BUS_~{INH}: track 66.7 -> 0.00 mm, vias 2 -> 0
- net /BUS_~{RES}: track 63.1 -> 0.00 mm, vias 2 -> 0
- net /BUS_~{DMAOUT}: track 59.6 -> 0.00 mm, vias 2 -> 0
- net /BUS_~{IRQ}: track 58.9 -> 0.00 mm, vias 2 -> 0
- net /C11: track 57.8 -> 0.00 mm
- net /BUS_~{INTOUT}: track 56.2 -> 0.00 mm, vias 2 -> 0
- net /C8: track 52.4 -> 0.00 mm
- net /C12: track 51.9 -> 0.00 mm
- net /B6: track 50.6 -> 0.00 mm, vias 1 -> 0
- net /C5: track 47.8 -> 0.00 mm
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
Commit message: final v5.3
Parts:
- added C11: C, Capacitor_SMD:C_0603_1608Metric, F.Cu at (159.0, 121.2)
- added C12: C, Capacitor_SMD:C_0603_1608Metric, F.Cu at (176.5, 121.8)
- added C14: C, Capacitor_SMD:C_0603_1608Metric, F.Cu at (202.2, 122.0)
- added C16: C, Capacitor_SMD:C_0603_1608Metric, F.Cu at (184.0, 121.5)
- added C18: C, Capacitor_SMD:C_0603_1608Metric, F.Cu at (132.0, 113.8)
- added C19: C, Capacitor_SMD:C_0603_1608Metric, F.Cu at (150.5, 114.2)
- moved R8 56.4 mm to (196.0, 84.0), turned to -90 degrees
- moved C17 55.2 mm to (194.2, 77.8), turned to 180 degrees
- moved R7 54.8 mm to (199.5, 84.0), turned to 90 degrees
- moved U8 53.6 mm to (199.2, 79.0)
- moved D1 53.3 mm to (185.5, 79.5), turned to 0 degrees
- moved R9 51.6 mm to (202.0, 84.0), turned to 90 degrees
- moved C5 19.0 mm to (132.0, 110.8), turned to 180 degrees
- moved R11 18.8 mm to (221.8, 75.2), turned to -90 degrees
- moved R13 18.0 mm to (201.2, 112.8), turned to 180 degrees
- moved R12 17.2 mm to (219.2, 75.2), turned to -90 degrees
- moved R14 13.8 mm to (205.0, 112.8), turned to 180 degrees
- moved C8 10.9 mm to (150.5, 111.2), turned to 0 degrees
- moved R15 10.6 mm to (209.0, 112.8), turned to 180 degrees
- moved U4 10.4 mm to (218.8, 84.2), turned to 90 degrees
- moved U3 10.1 mm to (193.0, 120.0)
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Connections:
- J1 pad 36: unconnected-(J1-Pin_36-Pad36) -> /BUS_7M
- J1 pad 37: unconnected-(J1-Pin_37-Pad37) -> /BUS_Q3
- J2 pad 1: /RAW -> unconnected-(J2-Pin_1-Pad1)
- J2 pad 19: +3V3 -> unconnected-(J2-Pin_19-Pad19)
- J3 pad 19: +3V3 -> unconnected-(J3-Pin_19-Pad19)
- J5 pad 2: unconnected-(J5-Pin_2-Pad2) -> /RAW
- R15 pad 2: /BUS_~{IRQ} -> /BUS_~{RDY}
- R18 pad 2: /BUS_~{RDY} -> /BUS_~{IRQ}
- U1 pad 13: /BUS_A0 -> GND
- U1 pad 14: /BUS_A1 -> GND
- U1 pad 16: /BUS_A2 -> GND
- U1 pad 17: /BUS_A3 -> GND
- U1 pad 19: /BUS_A4 -> GND
- U1 pad 20: /BUS_A5 -> GND
- U1 pad 22: /BUS_A6 -> GND
- U1 pad 23: /BUS_A7 -> /BUS_A0
- U1 pad 26: /A3 -> /C48
- U1 pad 27: /A6 -> GND
- U1 pad 29: /A9 -> GND
- U1 pad 30: /A12 -> GND
- U1 pad 32: /A2 -> GND
- U1 pad 33: /A5 -> GND
- U1 pad 35: /A8 -> GND
- U1 pad 36: /A11 -> GND
- U2 pad 11: /BUS_A14 -> /BUS_A7
- U2 pad 12: /BUS_A15 -> /BUS_A8
- U2 pad 13: /BUS_R~{W} -> /BUS_A9
- U2 pad 14: GND -> /BUS_A10
- U2 pad 16: GND -> /BUS_A11
- U2 pad 17: GND -> /BUS_A12
- U2 pad 19: GND -> /BUS_A13
- U2 pad 2: /BUS_A8 -> /BUS_A1
- U2 pad 20: GND -> /BUS_A14
- U2 pad 22: GND -> /BUS_A15
- U2 pad 23: GND -> /BUS_R~{W}
- U2 pad 26: GND -> /B46
- U2 pad 27: GND -> /B45
- U2 pad 29: GND -> /B49
- U2 pad 3: /BUS_A9 -> /BUS_A2
- U2 pad 30: GND -> /B48
- U2 pad 32: GND -> /A34
- U2 pad 33: GND -> /A33
- U2 pad 35: GND -> /A37
- U2 pad 37: /A39 -> /A40
- U2 pad 38: /A40 -> /A39
- U2 pad 40: /A42 -> /A43
- U2 pad 41: /A43 -> /A42
- U2 pad 43: /A45 -> /A46
- U2 pad 44: /A46 -> /A45
- U2 pad 46: /A48 -> /A49
- U2 pad 47: /A49 -> /A48
- U2 pad 5: /BUS_A10 -> /BUS_A3
- U2 pad 6: /BUS_A11 -> /BUS_A4
- U2 pad 8: /BUS_A12 -> /BUS_A5
- U2 pad 9: /BUS_A13 -> /BUS_A6
- U3 pad 11: /BUS_~{DMA} -> /BUS_~{RES}
- U3 pad 12: /BUS_~{INTIN} -> /BUS_~{IRQ}
- U3 pad 13: /BUS_~{DMAIN} -> /BUS_~{NMI}
- U3 pad 14: GND -> /BUS_~{RDY}
- U3 pad 16: GND -> /BUS_~{DMA}
- U3 pad 17: GND -> /BUS_~{INTIN}
- U3 pad 19: GND -> /BUS_~{DMAIN}
- U3 pad 30: GND -> /A23
- U3 pad 32: GND -> /B2
- U3 pad 33: GND -> /B3
- U3 pad 35: GND -> /B8
- U3 pad 36: /B39 -> /B11
- U3 pad 37: /B43 -> /B12
- U3 pad 38: /B42 -> /B40
- U3 pad 40: /B46 -> /B39
- U3 pad 41: /B45 -> /B9
- U3 pad 43: /B49 -> /B5
- U3 pad 44: /B48 -> /B6
- U3 pad 46: /A34 -> /B43
- U3 pad 47: /A33 -> /B42
- U3 pad 5: /BUS_M2B0 -> /BUS_Q3
- U3 pad 6: /BUS_~{INH} -> /BUS_7M
- U3 pad 8: /BUS_~{RES} -> /BUS_M2B0
- U3 pad 9: /BUS_~{IRQ} -> /BUS_~{INH}
- U4 pad 1: /B2 -> GND
- U4 pad 10: /~{OE} -> /BUS_~{INTOUT}
- U4 pad 11: /A37 -> /C40
- U4 pad 12: unconnected-(U4-Pad12) -> /~{OE}
- U4 pad 13: GND -> /C43
- U4 pad 2: /BUS_~{DMAOUT} -> unconnected-(U4-Pad2)
- U4 pad 3: /BUS_~{DMAIN} -> /BUS_~{INTIN}
- U4 pad 4: /BUS_~{DMAOUT} -> /BUS_~{INTOUT}
- U4 pad 5: /BUS_~{INTIN} -> /BUS_~{DMAIN}
- U4 pad 6: /BUS_~{INTOUT} -> /BUS_~{DMAOUT}
- U4 pad 8: /BUS_~{INTOUT} -> /BUS_~{DMAOUT}
- U4 pad 9: /A23 -> /C39
- U7 pad 1: /B5 -> /A14
- U7 pad 11: /B12 -> /A11
- U7 pad 12: /BUS_~{RDY} -> /BUS_~{IRQ}
- U7 pad 13: /B6 -> /A9
- U7 pad 3: /B8 -> /A15
- U7 pad 5: /B11 -> /A24
- U7 pad 6: /BUS_~{IRQ} -> /BUS_~{RDY}
- U7 pad 9: /B9 -> /A12
- U8 pad 4: /B40 -> /C42
Routing:
- net GND: track 0.00 -> 180.7 mm, vias 0 -> 55
- net /~{OE}: track 0.00 -> 152.2 mm, vias 0 -> 8
- net +5V: track 0.00 -> 150.0 mm, vias 0 -> 3
- net +3V3: track 0.00 -> 130.5 mm, vias 0 -> 13
- net /BUS_~{DMAIN}: track 0.00 -> 81.6 mm, vias 0 -> 2
- net /BUS_~{INTIN}: track 0.00 -> 80.7 mm, vias 0 -> 2
- net /C11: track 0.00 -> 73.0 mm
- net /BUS_~{INTOUT}: track 0.00 -> 71.9 mm, vias 0 -> 2
- net /BUS_~{DMAOUT}: track 0.00 -> 71.4 mm, vias 0 -> 2
- net /BUS_~{IRQ}: track 0.00 -> 69.8 mm, vias 0 -> 4
- net /BUS_~{DMA}: track 0.00 -> 69.3 mm, vias 0 -> 2
- net /BUS_~{NMI}: track 0.00 -> 67.2 mm, vias 0 -> 2
- net /BUS_~{INH}: track 0.00 -> 66.9 mm, vias 0 -> 3
- net /BUS_~{RES}: track 0.00 -> 64.8 mm, vias 0 -> 3
- net /C12: track 0.00 -> 64.6 mm
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
Commit message: v5 point
Parts:
- removed C17, C18, C19: C, Capacitor_SMD:C_0603_1608Metric
- added U5: 74LS245, Package_SO:TSSOP-20_4.4x6.5mm_P0.65mm, F.Cu at (181.5, 123.0)
- added U6: 74LS245, Package_SO:TSSOP-20_4.4x6.5mm_P0.65mm, F.Cu at (161.2, 123.5)
- added U9: 74LS245, Package_SO:TSSOP-20_4.4x6.5mm_P0.65mm, F.Cu at (216.0, 122.2)
- C1, C10, C11, C12, C13, C14, C16, C2, C3, C4, C6, C7, C8, C9: footprint Capacitor_SMD:C_0603_1608Metric -> Capacitor_SMD:C_0402_1005Metric
- C15, C5: footprint Capacitor_SMD:C_0603_1608Metric -> Capacitor_SMD:C_0805_2012Metric
- U1, U2, U3: value MC74LCX16245DT -> 74LS245; footprint Package_SO:TSSOP-48_6.1x12.5mm_P0.5mm -> Package_SO:TSSOP-20_4.4x6.5mm_P0.65mm
- moved C6 82.4 mm to (145.2, 127.0), turned to 0 degrees
- moved C11 62.1 mm to (221.0, 125.2), turned to 0 degrees
- moved C7 54.4 mm to (166.1, 126.4), turned to 0 degrees
- moved C12 48.1 mm to (196.0, 77.8), turned to 180 degrees
- moved C16 46.9 mm to (143.2, 98.2), turned to 90 degrees
- moved C14 42.6 mm to (214.5, 81.2), turned to 180 degrees
- moved C13 37.9 mm to (212.2, 93.5), turned to 90 degrees
- moved C8 29.8 mm to (176.2, 126.2)
- moved C9 28.5 mm to (186.5, 126.0), turned to 0 degrees
- moved C10 26.6 mm to (202.2, 125.5)
- moved C15 23.5 mm to (218.2, 136.2), turned to 90 degrees
- moved R13 16.9 mm to (199.2, 96.0), turned to 0 degrees
- moved R14 14.4 mm to (199.2, 99.5), turned to 0 degrees
- moved R15 14.3 mm to (199.2, 102.2), turned to 0 degrees
- moved C5 12.2 mm to (140.2, 101.8), turned to -90 degrees
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Connections:
- C13 pad 1: +3V3 -> +5V
- C14 pad 1: +3V3 -> +5V
- C15 pad 1: +3V3 -> +5V
- C6 pad 1: +5V -> +3V3
- C7 pad 1: +5V -> +3V3
- J4 pad 2: +3V3 -> unconnected-(J4-Pin_2-Pad2)
- R15 pad 2: /BUS_~{RDY} -> /BUS_~{IRQ}
- R18 pad 2: /BUS_~{IRQ} -> /BUS_~{RDY}
- U1 pad 1: /C48 -> /C3
- U1 pad 11: /BUS_D6 -> /BUS_D0
- U1 pad 12: /BUS_D7 -> /BUS_D1
- U1 pad 13: GND -> /BUS_D2
- U1 pad 14: GND -> /BUS_D3
- U1 pad 15: GND -> /BUS_D4
- U1 pad 16: GND -> /BUS_D5
- U1 pad 17: GND -> /BUS_D6
- U1 pad 18: +3V3 -> /BUS_D7
- U1 pad 19: GND -> /~{OE}
- U1 pad 2: /BUS_D0 -> /A2
- U1 pad 20: GND -> +3V3
- U1 pad 3: /BUS_D1 -> /A5
- U1 pad 4: GND -> /A8
- U1 pad 5: /BUS_D2 -> /A11
- U1 pad 6: /BUS_D3 -> /C40
- U1 pad 7: +3V3 -> /C43
- U1 pad 8: /BUS_D4 -> /C46
- U1 pad 9: /BUS_D5 -> /C49
- U2 pad 1: /C49 -> /C2
- U2 pad 11: /BUS_A7 -> /BUS_A8
- U2 pad 12: /BUS_A8 -> /BUS_A9
- U2 pad 13: /BUS_A9 -> /BUS_A10
- U2 pad 14: /BUS_A10 -> /BUS_A11
- U2 pad 15: GND -> /BUS_A12
- U2 pad 16: /BUS_A11 -> /BUS_A13
- U2 pad 17: /BUS_A12 -> /BUS_A14
- U2 pad 18: +3V3 -> /BUS_A15
- U2 pad 19: /BUS_A13 -> /~{OE}
- U2 pad 2: /BUS_A1 -> /A34
- U2 pad 20: /BUS_A14 -> +3V3
- U2 pad 3: /BUS_A2 -> /A33
- U2 pad 4: GND -> /A37
- U2 pad 5: /BUS_A3 -> /A36
- U2 pad 6: /BUS_A4 -> /A40
- U2 pad 7: +3V3 -> /A39
- U2 pad 8: /BUS_A5 -> /A43
- U2 pad 9: /BUS_A6 -> /A42
- U3 pad 11: /BUS_~{RES} -> /BUS_PHI0
- U3 pad 12: /BUS_~{IRQ} -> /BUS_M2SEL
- U3 pad 13: /BUS_~{NMI} -> /BUS_Q3
- U3 pad 14: /BUS_~{RDY} -> /BUS_7M
- U3 pad 15: GND -> /BUS_M2B0
- U3 pad 16: /BUS_~{DMA} -> /BUS_~{INH}
- U3 pad 17: /BUS_~{INTIN} -> /BUS_~{RES}
- U3 pad 18: +3V3 -> /BUS_~{IRQ}
- U3 pad 19: /BUS_~{DMAIN} -> /~{OE}
- U3 pad 2: /BUS_PHI0 -> /B40
- U3 pad 20: GND -> +3V3
- U3 pad 3: /BUS_M2SEL -> /B39
- U3 pad 4: GND -> /B43
- U3 pad 5: /BUS_Q3 -> /B42
- U3 pad 6: /BUS_7M -> /B46
- U3 pad 7: +3V3 -> /B45
- U3 pad 8: /BUS_M2B0 -> /B49
- U3 pad 9: /BUS_~{INH} -> /B48
- U4 pad 11: /C40 -> /C11
- U4 pad 13: /C43 -> /C12
- U7 pad 1: /A14 -> /B2
- U7 pad 11: /A11 -> /A23
- U7 pad 12: /BUS_~{IRQ} -> /BUS_~{RDY}
- U7 pad 13: /A9 -> /A14
- U7 pad 3: /A15 -> /B3
- U7 pad 5: /A24 -> /B5
- U7 pad 6: /BUS_~{RDY} -> /BUS_~{IRQ}
- U7 pad 9: /A12 -> /A24
- U8 pad 4: /C42 -> /C8
Routing:
- net GND: track 180.7 -> 23.2 mm, vias 55 -> 17
- net +3V3: track 130.5 -> 37.8 mm, vias 13 -> 10
- net /C9: track 57.0 -> 0.00 mm
- net /C2: track 45.9 -> 100.6 mm, vias 0 -> 3
- net /C5: track 54.6 -> 0.00 mm
- net /C48: track 48.5 -> 0.00 mm, vias 2 -> 0
- net /C6: track 47.0 -> 0.00 mm
- net /A8: track 0.00 -> 46.4 mm
- net /C42: track 42.3 -> 0.00 mm
- net /A5: track 0.00 -> 42.0 mm
- net /C46: track 0.00 -> 41.8 mm, vias 0 -> 1
- net /A2: track 0.00 -> 37.4 mm
- net /A9: track 60.8 -> 26.8 mm, vias 0 -> 1
- net /A12: track 57.8 -> 26.2 mm, vias 0 -> 1
- net /B6: track 18.1 -> 47.5 mm
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
Commit message: v5 board order
Parts:
- C1, C2: footprint Capacitor_SMD:C_0402_1005Metric -> Capacitor_SMD:C_0805_2012Metric
- C15, C5: footprint Capacitor_SMD:C_0805_2012Metric -> Capacitor_SMD:C_0402_1005Metric
- moved C13 74.9 mm to (145.2, 127.0), turned to 0 degrees
- moved C14 73.2 mm to (143.2, 98.2), turned to 90 degrees
- moved C16 73.2 mm to (214.5, 81.2), turned to 180 degrees
- moved C3 67.0 mm to (220.5, 136.8), turned to 90 degrees
- moved C2 64.9 mm to (140.2, 101.8), turned to -90 degrees
- moved C6 54.7 mm to (199.2, 135.8), turned to 90 degrees
- moved C15 43.2 mm to (212.2, 93.5)
- moved C5 38.6 mm to (153.5, 138.0), turned to 180 degrees
- moved C4 3.13 mm to (196.5, 134.2)
- moved C1 2.30 mm to (218.2, 136.2)
- moved C7 0.16 mm to (166.0, 126.2)
Connections:
- C13 pad 1: +5V -> +3V3
- C14 pad 1: +5V -> +3V3
- C16 pad 1: +3V3 -> +5V
- C2 pad 1: -5V -> +3V3
- C3 pad 1: +12V -> +5V
- C4 pad 1: -12V -> -5V
- C5 pad 1: +3V3 -> +12V
- C6 pad 1: +3V3 -> -12V
- J5 pad 1: unconnected-(J5-Pin_1-Pad1) -> GND
Routing:
- net GND: vias 17 -> 26
