File: v5/AppleTini_board/AppleTini_board.kicad_sch (KiCad schematic)
At the start: 12 parts, among them J1 Conn_02x25_Counter_Clockwise, J2 Conn_02x18_Odd_Even, J3 Conn_02x18_Odd_Even, J4 Conn_02x18_Odd_Even, J5 Conn_02x18_Odd_Even, U1 74LS245, U2 74LS245, U3 74LS245, U4 74LS245, U5 74LS245, U6 74LS245, U7 74LCX07

Commit message: v5 first draftw
Parts:
- removed J2, J3, J4, J5: Conn_02x18_Odd_Even, symbol Connector_Generic:Conn_02x18_Odd_Even
- removed U1, U2, U3, U4, U5, U6: 74LS245, symbol 74xx:74LS245
- added C1, C10, C11, C12, C13, C14, C15, C16, C17, C2, C3, C4, C5, C6, C7, C8, C9: C, Capacitor_SMD:C_0603_1608Metric, symbol Device:C
- added J2, J3: Conn_02x14_Odd_Even, Connector_PinHeader_2.54mm:PinHeader_2x14_P2.54mm_Vertical, symbol Connector_Generic:Conn_02x14_Odd_Even
- added J4, J5: Conn_02x05_Odd_Even, Connector_PinHeader_2.54mm:PinHeader_2x05_P2.54mm_Vertical, symbol Connector_Generic:Conn_02x05_Odd_Even
- added R1, R10, R11, R12, R2, R3, R4, R5, R6, R7, R8, R9: R_US, Resistor_SMD:R_0402_1005Metric, symbol Device:R_US
- added U1, U2, U3: MC74LCX16245DT, Package_SO:TSSOP-48_6.1x12.5mm_P0.5mm, symbol 74xx:MC74LCX16245DT
- added U8: 74LVC1G04, Package_TO_SOT_SMD:SOT-23-5, symbol 74xGxx:74LVC1G04
- U7: footprint (none) -> Package_SO:TSSOP-14_4.4x5mm_P0.65mm
Connections:
- net +12V: now also C3.1
- net +5V: now also C1.1, R7.1, R9.1
- net -12V: now also C4.1
- net -5V: now also C2.1
- net BUS_A0: now also U1.13 (B8)
- net BUS_A1: now also U1.14 (B9)
- net BUS_A10: now also U2.5 (B2)
- net BUS_A11: now also U2.6 (B3)
- net BUS_A12: now also U2.8 (B4)
- net BUS_A13: now also U2.9 (B5)
- net BUS_A14: now also U2.11 (B6)
- net BUS_A15: now also U2.12 (B7)
- net BUS_A2: now also U1.16 (B10)
- net BUS_A3: now also U1.17 (B11)
- net BUS_A4: now also U1.19 (B12)
- net BUS_A5: now also U1.20 (B13)
- net BUS_A6: now also U1.22 (B14)
- net BUS_A7: now also U1.23 (B15)
- net BUS_A8: now also U2.2 (B0)
- net BUS_A9: now also U2.3 (B1)
- net BUS_D0: now also U1.2 (B0)
- net BUS_D1: now also U1.3 (B1)
- net BUS_D2: now also U1.5 (B2)
- net BUS_D3: now also U1.6 (B3)
- net BUS_D4: now also U1.8 (B4)
- net BUS_D5: now also U1.9 (B5)
- net BUS_D6: now also U1.11 (B6)
- net BUS_D7: now also U1.12 (B7)
- net BUS_M2B0: now also U3.5 (B2)
- net BUS_M2SEL: now also U3.3 (B1)
- net BUS_PHI0: now also U3.2 (B0)
- net BUS_R~{W}: now also U2.13 (B8)
- net BUS_~{DMAIN}: now also U3.13 (B8)
- net BUS_~{DMAOUT}: now also U7.12, R12.2; no longer U7.2
- net BUS_~{DMA}: now also U7.8, U3.11 (B6); no longer U7.6
- net BUS_~{INH}: now also U7.2, U3.6 (B3); no longer U7.12
- net BUS_~{INTIN}: now also U3.12 (B7)
- net BUS_~{INTOUT}: now also U7.10, R11.2; no longer U7.4
- net BUS_~{IRQ}: now also U7.6, U3.9 (B5)
- net BUS_~{RES}: now also U7.4, U3.8 (B4); no longer U7.8
- net GND: now also U7.7 (GND), C1.2, C10.2, C11.2, C12.2, C13.2, C14.2, C15.2, C16.2, C17.2, C2.2, C3.2, C4.2, C5.2, C6.2, C7.2, C8.2, C9.2, J2.2 (Pin_2), J2.20 (Pin_20), J3.2 (Pin_2), J3.20 (Pin_20), J4.1 (Pin_1), R8.2, U1.10 (GND), U1.15 (GND), U1.21 (GND), U1.28 (GND), U1.34 (GND), U1.39 (GND), U1.4 (GND), U1.45 (GND), U2.10 (GND), U2.14 (B9), U2.15 (GND), U2.16 (B10), U2.17 (B11), U2.19 (B12), U2.20 (B13), U2.21 (GND), U2.22 (B14), U2.23 (B15), U2.26 (A15), U2.27 (A14), U2.28 (GND), U2.29 (A13), U2.30 (A12), U2.32 (A11), U2.33 (A10), U2.34 (GND), U2.35 (A9), U2.39 (GND), U2.4 (GND), U2.45 (GND), U3.1 (T/~{R}1), U3.10 (GND), U3.14 (B9), U3.15 (GND), U3.16 (B10), U3.17 (B11), U3.19 (B12), U3.20 (B13), U3.21 (GND), U3.22 (B14), U3.23 (B15), U3.24 (T/~{R}2), U3.26 (A15), U3.27 (A14), U3.28 (GND), U3.29 (A13), U3.30 (A12), U3.32 (A11), U3.33 (A10), U3.34 (GND), U3.35 (A9), U3.39 (GND), U3.4 (GND), U3.45 (GND), U8.3 (GND)
- net +3V3: now reaches U7.14 (VCC)
- net +3V3: now also C10.1, C11.1, C12.1, C13.1, C14.1, C15.1, C16.1, C17.1, C5.1, C6.1, C7.1, C8.1, C9.1, J2.19 (Pin_19), J3.1 (Pin_1), J3.19 (Pin_19), J4.2 (Pin_2), R1.1, R10.1, R11.1, R12.1, R2.1, R3.1, R4.1, R5.1, R6.1, U1.18 (VCC), U1.31 (VCC), U1.42 (VCC), U1.7 (VCC), U2.18 (VCC), U2.31 (VCC), U2.42 (VCC), U2.7 (VCC), U3.18 (VCC), U3.31 (VCC), U3.42 (VCC), U3.7 (VCC), U8.5 (VCC)
- net B11: now reaches U7.5
- net B11: now also J3.28 (Pin_28), R3.2
- net B8: now reaches U7.3
- net B8: now also J3.26 (Pin_26), R2.2
- net B9: now reaches U7.9
- net B9: now also J3.25 (Pin_25), R4.2
- net B12: now reaches U7.11
- net B12: now also J3.27 (Pin_27), R5.2
- net B6: now reaches U7.13
- net B6: now also J3.23 (Pin_23), R6.2
- net B5: now reaches U7.1
- net B5: now also J3.24 (Pin_24), R1.2
- net BUS_~{RDY}: no longer names the net of J1.21 (Pin_21)
- net BUS_~{RDY}: no longer U7.10
- new net: R7.2, R8.1, R9.2, U8.2
- new net A11: J3.10 (Pin_10), U1.36 (A8)
- new net A12: J3.9 (Pin_9), U1.30 (A12)
- new net A14: J3.12 (Pin_12)
- new net A15: J3.11 (Pin_11)
- new net A17: J3.14 (Pin_14)
- new net A18: J3.13 (Pin_13)
- new net A2: J3.4 (Pin_4), U1.32 (A11)
- new net A20: J3.16 (Pin_16)
- new net A21: J3.15 (Pin_15)
- new net A23: J3.18 (Pin_18)
- new net A24: J3.17 (Pin_17)
- new net A27: J2.17 (Pin_17)
- new net A28: J2.18 (Pin_18)
- new net A3: J3.3 (Pin_3), U1.26 (A15)
- new net A30: J2.15 (Pin_15)
- new net A31: J2.16 (Pin_16)
- new net A33: J2.13 (Pin_13), U3.47 (A0)
- new net A34: J2.14 (Pin_14), U3.46 (A1)
- new net A36: J2.11 (Pin_11), U2.36 (A8)
- new net A37: J2.12 (Pin_12), R10.2, U1.25 (~{OE2}), U1.48 (~{OE1}), U2.25 (~{OE2}), U2.48 (~{OE1}), U3.25 (~{OE2}), U3.48 (~{OE1})
- new net A39: J2.9 (Pin_9), U2.37 (A7)
- new net A40: J2.10 (Pin_10), U2.38 (A6)
- new net A42: J2.7 (Pin_7), U2.40 (A5)
- new net A43: J2.8 (Pin_8), U2.41 (A4)
- new net A45: J2.5 (Pin_5), U2.43 (A3)
- new net A46: J2.6 (Pin_6), U2.44 (A2)
- new net A48: J2.3 (Pin_3), U2.46 (A1)
- new net A49: J2.4 (Pin_4), U2.47 (A0)
- new net A5: J3.6 (Pin_6), U1.33 (A10)
- new net A6: J3.5 (Pin_5), U1.27 (A14)
- new net A8: J3.8 (Pin_8), U1.35 (A9)
- new net A9: J3.7 (Pin_7), U1.29 (A13)
- new net B2: J3.22 (Pin_22)
- new net B3: J3.21 (Pin_21)
- new net B39: J2.27 (Pin_27), U3.36 (A8)
- new net B40: J2.28 (Pin_28), U8.4
- new net B42: J2.25 (Pin_25), U3.38 (A6)
- new net B43: J2.26 (Pin_26), U3.37 (A7)
- new net B45: J2.23 (Pin_23), U3.41 (A4)
- new net B46: J2.24 (Pin_24), U3.40 (A5)
- new net B48: J2.21 (Pin_21), U3.44 (A2)
- new net B49: J2.22 (Pin_22), U3.43 (A3)
- new net C11: J5.9 (Pin_9), U1.47 (A0)
- new net C12: J5.10 (Pin_10), U1.46 (A1)
- new net C2: J5.3 (Pin_3), U1.38 (A6)
- new net C3: J5.4 (Pin_4), U1.37 (A7)
- new net C39: J4.10 (Pin_10)
- new net C40: J4.9 (Pin_9)
- new net C42: J4.8 (Pin_8)
- new net C43: J4.7 (Pin_7)
- new net C45: J4.6 (Pin_6)
- new net C46: J4.5 (Pin_5)
- new net C48: J4.4 (Pin_4), U1.1 (T/~{R}1)
- new net C49: J4.3 (Pin_3), U1.24 (T/~{R}2), U2.1 (T/~{R}1), U2.24 (T/~{R}2)
- new net C5: J5.5 (Pin_5), U1.41 (A4)
- new net C6: J5.6 (Pin_6), U1.40 (A5)
- new net C8: J5.7 (Pin_7), U1.44 (A2)
- new net C9: J5.8 (Pin_8), U1.43 (A3)
- new net RAW: J2.1 (Pin_1)
- no-connect marks 8 -> 18
Other:
- moved on the sheet: U7A, U7B, U7C, U7D, U7E, U7F, U7G

Commit message: wip, reworking
Parts:
- removed C11, C12, C14, C16: C, Capacitor_SMD:C_0603_1608Metric, symbol Device:C
- removed R10, R2, R3, R4, R5, R6: R_US, Resistor_SMD:R_0402_1005Metric, symbol Device:R_US
- added D1: D_Schottky, Diode_SMD:Nexperia_CFP3_SOD-123W, symbol Device:D_Schottky
- added R13, R14, R15, R16, R17, R18: R_US, Resistor_SMD:R_0402_1005Metric, symbol Device:R_US
- added U4: 74LCX07, Package_SO:TSSOP-14_4.4x5mm_P0.65mm, symbol 74xx:74LCX07
- C1, C10, C13, C15, C17, C2, C3, C4, C5, C6, C7, C8, C9: LCSC (none) -> C14663
- J2, J3, J4, J5: now not fitted
- R1, R11, R12, R7, R8, R9: LCSC (none) -> C2991755
- U1, U2, U3: LCSC (none) -> C7824
- U7: LCSC (none) -> C2676034
- U8: JCSC (none) -> C7827
Connections:
- net +3V3: no longer C6.1, C7.1, R1.1, R11.1, R12.1, U7.14 (VCC)
- net +5V: now also C6.1, C7.1, R1.1, R11.1, R12.1, U7.14 (VCC), D1.2 (A), R13.1, R14.1, R15.1, R16.1, R17.1, R18.1, U4.14 (VCC)
- net A23: now also U4.9
- net A37: now also U4.11; no longer U1.25 (~{OE2}), U1.48 (~{OE1}), U2.25 (~{OE2}), U2.48 (~{OE1}), U3.25 (~{OE2}), U3.48 (~{OE1})
- net B2: now also U4.1
- net B5: no longer R1.2
- net BUS_~{DMAIN}: now also U4.3
- net BUS_~{DMAOUT}: now also R11.2, U4.2, U4.4; no longer R12.2, U7.12
- net BUS_~{DMA}: now also R16.2
- net BUS_~{INH}: now also R13.2
- net BUS_~{INTIN}: now also U4.5
- net BUS_~{INTOUT}: now also R12.2, U4.6, U4.8; no longer R11.2, U7.10
- net BUS_~{IRQ}: now also R15.2
- net BUS_~{RES}: now also R14.2
- net GND: now also U4.13, U4.7 (GND)
- net RAW: now also D1.1 (K)
- net BUS_~{RDY}: now reaches J1.21 (Pin_21)
- net BUS_~{RDY}: now also U7.12, R18.2
- net BUS_~{NMI}: now reaches J1.29 (Pin_29)
- net BUS_~{NMI}: now also U7.10, R17.2
- new net ~{OE}: R1.2, U1.25 (~{OE2}), U1.48 (~{OE1}), U2.25 (~{OE2}), U2.48 (~{OE1}), U3.25 (~{OE2}), U3.48 (~{OE1}), U4.10
- no-connect marks 18 -> 16
Other:
- moved on the sheet: C10, C13, C15, C17, C6, C7, C9, U7A, U7B, U7D, U7E

Commit message: final v5.3
Parts:
- added C11, C12, C14, C16, C18, C19: C, Capacitor_SMD:C_0603_1608Metric, symbol Device:C
Connections:
- net +3V3: now also C11.1, C12.1, C14.1, C16.1, C18.1, C19.1; no longer J2.19 (Pin_19), J3.19 (Pin_19)
- net A11: now also U7.11; no longer U1.36 (A8)
- net A12: now also U7.9; no longer U1.30 (A12)
- net A14: now also U7.1
- net A15: now also U7.3
- net A2: no longer U1.32 (A11)
- net A23: now also U3.30 (A12); no longer U4.9
- net A24: now also U7.5
- net A3: no longer U1.26 (A15)
- net A33: now also U2.33 (A10); no longer U3.47 (A0)
- net A34: now also U2.32 (A11); no longer U3.46 (A1)
- net A37: now also U2.35 (A9); no longer U4.11
- net A39: now also U2.38 (A6); no longer U2.37 (A7)
- net A40: now also U2.37 (A7); no longer U2.38 (A6)
- net A42: now also U2.41 (A4); no longer U2.40 (A5)
- net A43: now also U2.40 (A5); no longer U2.41 (A4)
- net A45: now also U2.44 (A2); no longer U2.43 (A3)
- net A46: now also U2.43 (A3); no longer U2.44 (A2)
- net A48: now also U2.47 (A0); no longer U2.46 (A1)
- net A49: now also U2.46 (A1); no longer U2.47 (A0)
- net A5: no longer U1.33 (A10)
- net A6: no longer U1.27 (A14)
- net A8: no longer U1.35 (A9)
- net A9: now also U7.13; no longer U1.29 (A13)
- net B11: now also U3.36 (A8); no longer U7.5
- net B12: now also U3.37 (A7); no longer U7.11
- net B2: now also U3.32 (A11); no longer U4.1
- net B3: now also U3.33 (A10)
- net B39: now also U3.40 (A5); no longer U3.36 (A8)
- net B40: now also U3.38 (A6); no longer U8.4
- net B42: now also U3.47 (A0); no longer U3.38 (A6)
- net B43: now also U3.46 (A1); no longer U3.37 (A7)
- net B45: now also U2.27 (A14); no longer U3.41 (A4)
- net B46: now also U2.26 (A15); no longer U3.40 (A5)
- net B48: now also U2.30 (A12); no longer U3.44 (A2)
- net B49: now also U2.29 (A13); no longer U3.43 (A3)
- net B5: now also U3.43 (A3); no longer U7.1
- net B6: now also U3.44 (A2); no longer U7.13
- net B8: now also U3.35 (A9); no longer U7.3
- net B9: now also U3.41 (A4); no longer U7.9
- net BUS_A0: now also U1.23 (B15); no longer U1.13 (B8)
- net BUS_A1: now also U2.2 (B0); no longer U1.14 (B9)
- net BUS_A10: now also U2.14 (B9); no longer U2.5 (B2)
- net BUS_A11: now also U2.16 (B10); no longer U2.6 (B3)
- net BUS_A12: now also U2.17 (B11); no longer U2.8 (B4)
- net BUS_A13: now also U2.19 (B12); no longer U2.9 (B5)
- net BUS_A14: now also U2.20 (B13); no longer U2.11 (B6)
- net BUS_A15: now also U2.22 (B14); no longer U2.12 (B7)
- net BUS_A2: now also U2.3 (B1); no longer U1.16 (B10)
- net BUS_A3: now also U2.5 (B2); no longer U1.17 (B11)
- net BUS_A4: now also U2.6 (B3); no longer U1.19 (B12)
- net BUS_A5: now also U2.8 (B4); no longer U1.20 (B13)
- net BUS_A6: now also U2.9 (B5); no longer U1.22 (B14)
- net BUS_A7: now also U2.11 (B6); no longer U1.23 (B15)
- net BUS_A8: now also U2.12 (B7); no longer U2.2 (B0)
- net BUS_A9: now also U2.13 (B8); no longer U2.3 (B1)
- net BUS_M2B0: now also U3.8 (B4); no longer U3.5 (B2)
- net BUS_R~{W}: now also U2.23 (B15); no longer U2.13 (B8)
- net BUS_~{DMAIN}: now also U3.19 (B12), U4.5; no longer U3.13 (B8), U4.3
- net BUS_~{DMAOUT}: now also U4.6, U4.8; no longer U4.2, U4.4
- net BUS_~{DMA}: now also U3.16 (B10); no longer U3.11 (B6)
- net BUS_~{INH}: now also U3.9 (B5); no longer U3.6 (B3)
- net BUS_~{INTIN}: now also U3.17 (B11), U4.3; no longer U3.12 (B7), U4.5
- net BUS_~{INTOUT}: now also U4.10, U4.4; no longer U4.6, U4.8
- net BUS_~{IRQ}: now also R18.2, U3.12 (B7), U7.12; no longer R15.2, U3.9 (B5), U7.6
- net BUS_~{NMI}: now also U3.13 (B8)
- net BUS_~{RDY}: now also R15.2, U3.14 (B9), U7.6; no longer R18.2, U7.12
- net BUS_~{RES}: now also U3.11 (B6); no longer U3.8 (B4)
- net C39: now also U4.9
- net C40: now also U4.11
- net C42: now also U8.4
- net C43: now also U4.13
- net C48: now also U1.26 (A15)
- net GND: now also U1.13 (B8), U1.14 (B9), U1.16 (B10), U1.17 (B11), U1.19 (B12), U1.20 (B13), U1.22 (B14), U1.27 (A14), U1.29 (A13), U1.30 (A12), U1.32 (A11), U1.33 (A10), U1.35 (A9), U1.36 (A8), U4.1, C11.2, C12.2, C14.2, C16.2, C18.2, C19.2; no longer U2.14 (B9), U2.16 (B10), U2.17 (B11), U2.19 (B12), U2.20 (B13), U2.22 (B14), U2.23 (B15), U2.26 (A15), U2.27 (A14), U2.29 (A13), U2.30 (A12), U2.32 (A11), U2.33 (A10), U2.35 (A9), U3.14 (B9), U3.16 (B10), U3.17 (B11), U3.19 (B12), U3.30 (A12), U3.32 (A11), U3.33 (A10), U3.35 (A9), U4.13
- net RAW: now also J5.2 (Pin_2); no longer J2.1 (Pin_1)
- net ~{OE}: now also U4.12; no longer U4.10
- net BUS_7M: now reaches J1.36 (Pin_36)
- net BUS_7M: now also U3.6 (B3)
- net BUS_Q3: now reaches J1.37 (Pin_37)
- net BUS_Q3: now also U3.5 (B2)
- no-connect marks 16 -> 17
Other:
- moved on the sheet: J2, J3, J4, J5, R11, R12

Commit message: v5 point
Parts:
- removed C17, C18, C19, C5: C, Capacitor_SMD:C_0603_1608Metric, symbol Device:C
- removed U1, U2, U3: MC74LCX16245DT, Package_SO:TSSOP-48_6.1x12.5mm_P0.5mm, symbol 74xx:MC74LCX16245DT
- added C14: C, Capacitor_SMD:C_0402_1005Metric, symbol Device:C
- added U1, U2, U3, U5, U6, U9: 74LS245, Package_SO:TSSOP-20_4.4x6.5mm_P0.65mm, symbol 74xx:74LS245
- C1, C10, C11, C12, C13, C16, C2, C3, C4, C6, C7, C8, C9: footprint Capacitor_SMD:C_0603_1608Metric -> Capacitor_SMD:C_0402_1005Metric
- C15: footprint Capacitor_SMD:C_0603_1608Metric -> Capacitor_SMD:C_0805_2012Metric; LCSC C14663 -> (none)
- C5: renamed from C14; footprint Capacitor_SMD:C_0603_1608Metric -> Capacitor_SMD:C_0805_2012Metric
Connections:
- net +3V3: now also C6.1, C7.1, U1.20 (VCC), U2.20 (VCC), U3.20 (VCC), U5.20 (VCC), U6.20 (VCC), U9.20 (VCC); no longer C13.1, C15.1, J4.2 (Pin_2)
- net +5V: now also C13.1, C15.1, C14.1; no longer C6.1, C7.1
- net A11: now also U1.5 (A3); no longer U7.11
- net A12: now also U6.6 (A4); no longer U7.9
- net A14: now also U7.13; no longer U7.1
- net A15: now also U5.9 (A7); no longer U7.3
- net A2: now also U1.2 (A0)
- net A23: now also U7.11
- net A24: now also U7.9; no longer U7.5
- net A3: now also U6.9 (A7)
- net A33: now also U2.3 (A1)
- net A34: now also U2.2 (A0)
- net A36: now also U2.5 (A3)
- net A37: now also U2.4 (A2)
- net A39: now also U2.7 (A5)
- net A40: now also U2.6 (A4)
- net A42: now also U2.9 (A7)
- net A43: now also U2.8 (A6)
- net A45: now also U6.3 (A1)
- net A46: now also U6.2 (A0)
- net A48: now also U6.5 (A3)
- net A49: now also U6.4 (A2)
- net A5: now also U1.3 (A1)
- net A6: now also U6.8 (A6)
- net A8: now also U1.4 (A2)
- net A9: now also U6.7 (A5); no longer U7.13
- net B11: now also U9.6 (A4)
- net B12: now also U9.7 (A5)
- net B2: now also U7.1
- net B3: now also U7.3
- net B39: now also U3.3 (A1)
- net B40: now also U3.2 (A0)
- net B42: now also U3.5 (A3)
- net B43: now also U3.4 (A2)
- net B45: now also U3.7 (A5)
- net B46: now also U3.6 (A4)
- net B48: now also U3.9 (A7)
- net B49: now also U3.8 (A6)
- net B5: now also U7.5
- net B6: now also U9.9 (A7)
- net B8: now also U9.5 (A3)
- net B9: now also U9.8 (A6)
- net BUS_7M: now also U3.14 (B4)
- net BUS_A0: now also U6.11 (B7)
- net BUS_A1: now also U6.12 (B6)
- net BUS_A10: now also U2.13 (B5)
- net BUS_A11: now also U2.14 (B4)
- net BUS_A12: now also U2.15 (B3)
- net BUS_A13: now also U2.16 (B2)
- net BUS_A14: now also U2.17 (B1)
- net BUS_A15: now also U2.18 (B0)
- net BUS_A2: now also U6.13 (B5)
- net BUS_A3: now also U6.14 (B4)
- net BUS_A4: now also U6.15 (B3)
- net BUS_A5: now also U6.16 (B2)
- net BUS_A6: now also U6.17 (B1)
- net BUS_A7: now also U6.18 (B0)
- net BUS_A8: now also U2.11 (B7)
- net BUS_A9: now also U2.12 (B6)
- net BUS_D0: now also U1.11 (B7)
- net BUS_D1: now also U1.12 (B6)
- net BUS_D2: now also U1.13 (B5)
- net BUS_D3: now also U1.14 (B4)
- net BUS_D4: now also U1.15 (B3)
- net BUS_D5: now also U1.16 (B2)
- net BUS_D6: now also U1.17 (B1)
- net BUS_D7: now also U1.18 (B0)
- net BUS_M2B0: now also U3.15 (B3)
- net BUS_M2SEL: now also U3.12 (B6)
- net BUS_PHI0: now also U3.11 (B7)
- net BUS_Q3: now also U3.13 (B5)
- net BUS_R~{W}: now also U5.11 (B7)
- net BUS_~{DMAIN}: now also U9.15 (B3)
- net BUS_~{DMA}: now also U9.13 (B5)
- net BUS_~{INH}: now also U3.16 (B2)
- net BUS_~{INTIN}: now also U9.14 (B4)
- net BUS_~{IRQ}: now also R15.2, U7.6, U3.18 (B0); no longer R18.2, U7.12
- net BUS_~{NMI}: now also U9.11 (B7)
- net BUS_~{RDY}: now also R18.2, U7.12, U9.12 (B6); no longer R15.2, U7.6
- net BUS_~{RES}: now also U3.17 (B1)
- net C11: now also U4.11
- net C12: now also U4.13
- net C2: now also U2.1 (A->B), U5.1 (A->B), U6.1 (A->B)
- net C3: now also U1.1 (A->B)
- net C40: now also U1.6 (A4); no longer U4.11
- net C42: no longer U8.4
- net C43: now also U1.7 (A5); no longer U4.13
- net C46: now also U1.8 (A6)
- net C49: now also U1.9 (A7)
- net C8: now also U8.4
- net GND: now also C14.2, U1.10 (GND), U2.10 (GND), U3.1 (A->B), U3.10 (GND), U5.10 (GND), U5.12 (B6), U5.13 (B5), U5.14 (B4), U5.15 (B3), U5.16 (B2), U5.17 (B1), U5.18 (B0), U5.2 (A0), U5.3 (A1), U5.4 (A2), U5.5 (A3), U5.6 (A4), U5.7 (A5), U5.8 (A6), U6.10 (GND), U9.1 (A->B), U9.10 (GND), U9.16 (B2), U9.17 (B1), U9.18 (B0), U9.2 (A0), U9.3 (A1), U9.4 (A2)
- net ~{OE}: now also U1.19 (CE), U2.19 (CE), U3.19 (CE), U5.19 (CE), U6.19 (CE), U9.19 (CE)
- no-connect marks 17 -> 18
Other:
- moved on the sheet: C5, R11, R12, U4B, U4C, U4D, U4E

Commit message: v5 board order
Parts:
- C1: renamed from C15; LCSC (none) -> C440198
- C10: renamed from C8; LCSC C14663 -> C77177
- C11: renamed from C9; LCSC C14663 -> C77177
- C12: renamed from C10; LCSC C14663 -> C77177
- C13: renamed from C11; LCSC C14663 -> C77177
- C14: renamed from C12; LCSC C14663 -> C77177
- C15: renamed from C13; LCSC C14663 -> C77177
- C16: renamed from C14; LCSC C14663 -> C77177
- C2: renamed from C5; LCSC C14663 -> C440198
- C3: renamed from C1; LCSC C14663 -> C77177
- C4: renamed from C2; LCSC C14663 -> C77177
- C5: renamed from C3; LCSC C14663 -> C77177
- C6: renamed from C4; LCSC C14663 -> C77177
- C7: renamed from C16; LCSC C14663 -> C77177
- C8: renamed from C6; LCSC C14663 -> C77177
- C9: renamed from C7; LCSC C14663 -> C77177
- U1, U2, U3, U5, U6, U9: LCSC (none) -> C6082
Connections:
- net GND: now also J5.1 (Pin_1)
Other:
- moved on the sheet: C1, C14, C15, C16, C2, C3, C4, C5, C6, C7

Commit message: v5.1 Kicad design, v5.1 Alchitry design
Parts:
- removed C16: C, Capacitor_SMD:C_0402_1005Metric, symbol Device:C
- removed R11, R12, R13, R14, R15, R16, R17, R18: R_US, Resistor_SMD:R_0402_1005Metric, symbol Device:R_US
- removed U4, U7: 74LCX07, Package_SO:TSSOP-14_4.4x5mm_P0.65mm, symbol 74xx:74LCX07
- removed U9: 74LS245, Package_SO:TSSOP-20_4.4x6.5mm_P0.65mm, symbol 74xx:74LS245
- added R2: R_US, Resistor_SMD:R_0402_1005Metric, symbol Device:R_US
- added U4: TXS0108EPWR, Package_SO:TSSOP-20_4.4x6.5mm_P0.65mm, symbol Logic_LevelTranslator:TXS0108EPW
- C10, C11, C12, C13, C14, C15, C3, C4, C5, C6, C7, C8, C9: LCSC C77177 -> C77020
- U8: value 74LVC1G04 -> 74LVC1G04DBVRG
Connections:
- net BUS_~{DMAOUT} is gone; now on net BUS_~{DMAINOUT}: J1.24 (Pin_24)
- net BUS_~{INTOUT} is gone; now on net BUS_~{INTINOUT}: J1.23 (Pin_23)
- net ~{OE} is gone; now on net C11: R1.2, U1.19 (CE), U2.19 (CE), U3.19 (CE), U5.19 (CE), U6.19 (CE)
- net +3V3: now also R1.1, U4.2 (VCCA)
- net +5V: now also U4.19 (VCCB); no longer R1.1
- net A14: now also U4.4 (A3)
- net A23: now also U4.6 (A5)
- net A24: now also U4.5 (A4)
- net B2: now also U4.8 (A7)
- net B3: now also U4.7 (A6)
- net B39: no longer U3.3 (A1)
- net B40: no longer U3.2 (A0)
- net B43: no longer U3.4 (A2)
- net B5: now also U4.9 (A8)
- net BUS_~{DMA}: now also U4.17 (B3)
- net BUS_~{INH}: now also U4.12 (B8); no longer U3.16 (B2)
- net BUS_~{IRQ}: now also U4.14 (B6); no longer U3.18 (B0)
- net BUS_~{NMI}: now also U4.16 (B4)
- net BUS_~{RDY}: now also U4.15 (B5)
- net BUS_~{RES}: now also U4.13 (B7); no longer U3.17 (B1)
- net C12: now also R2.1, U4.10 (OE)
- net GND: now also U3.16 (B2), U3.17 (B1), U3.18 (B0), R2.2, U4.11 (GND)
- net BUS_~{DMAIN} renamed BUS_~{DMAINOUT}
- net BUS_~{INTIN} renamed BUS_~{INTINOUT}
- no-connect marks 18 -> 24
Other:
- moved on the sheet: R7, R8, R9, U8
